File: eagle/Controller-Power.sch (EAGLE design)
At the start: 24 parts, among them IC3 7818TV, X1 MKDSN1,5/2-5,08, X2 MKDSN1,5/2-5,08, X3 MKDSN1,5/2-5,08

Commit message: Lots of schema and board changes
Parts:
- removed C1, C7: 100nF, rcl:C-EUC0805
- removed C2, C8: 100µ, rcl:CPOL-EUE3.5-8
- removed D1, D3: 1N4004, diode:1N4004
- removed IC1: (no value), v-reg:LM317TS
- removed IC3: 7818TV, linear:7805TV
- removed JP2, JP3, JP4: (no value), pinhead:PINHD-1X2
- removed R1, R20: 100k, rcl:R-EU_R1206
- removed R2, R21: (no value), pot:TRIM_EU-PT10
- removed U$2: GLEICHRICHTER, Gleichrichter:GLEICHRICHTER
- removed X1, X2, X3: MKDSN1,5/2-5,08, con-phoenix-508:MKDSN1,5/2-5,08
- added TR1: (no value), trafo:EI38-1
- added U$1: GLEICHRICHTER, Gleichrichter:GLEICHRICHTER
- added X4: MKDSN1,5/2-5,08, con-phoenix-508:MKDSN1,5/2-5,08
- IC2: value (none) -> DCDC-WANDLER; device v-reg:LM317TS -> 0liver:DCDC-WANDLER
Connections:
- removed net N$2: C6.1, IC3.VO, JP4.1
- removed net N$24: U$2.AC1, X1-2.KL
- removed net N$28: D3.A, IC1.OUT, R20.2, X2-2.KL
- removed net N$29: JP1.2, R21.A
- removed net N$3: D1.A, IC2.OUT, R1.2, X3-2.KL
- removed net N$30: IC1.ADJ, JP1.1, R20.1
- removed net N$4: IC2.ADJ, JP2.1, R1.1
- removed net N$5: JP2.2, R2.A
- new net N$19: TR1.P1, X4-1.KL
- new net N$20: TR1.P2, X4-2.KL
- new net N$21: TR1.S3, U$1.AC2
- new net N$22: TR1.S4, U$1.AC1
- net GND: now also IC2.GND, JP1.2, U$1.-; no longer C1.2, C2.-, C7.2, C8.-, IC3.GND, JP3.1, JP3.2, JP4.2, R2.E, R2.S, R21.E, R21.S, U$2.-, X2-1.KL, X3-1.KL
- net N$17: now also IC2.VI, U$1.+; no longer C1.1, C2.+, C7.1, C8.+, D1.C, D3.C, IC1.IN, IC2.IN, IC3.VI, U$2.+
- net N$25: now also C6.1, IC2.VO, JP1.1; no longer U$2.AC2, X1-1.KL
Other:
- moved on the sheet: C4, C5, C6, JP1
